File: PCB/_autosave-spymic.kicad_sch (KiCad schematic)
At the start: 7 parts, among them J1 Conn_01x02_Pin, U1 GS8331-TR

Commit message: c ommit
Parts:
- removed R4: R_Variable, symbol Device:R_Variable
- added C1, C2, C3, C8, C9: 10uF, symbol Device:C_Polarized
- added C4, C6, C7: 10uF, symbol Device:C
- added C5: 22uF, symbol Device:C
- added CN1: PJ-320D, easyeda2kicad:AUDIO-SMD_PJ-320D-1, symbol LCSC:PJ-320D
- added R4, R6: 470, symbol Device:R
- added R5: RK09K1130A5R, easyeda2kicad:RES-ADJ-TH_RK09K1130A5R, symbol LCSC:RK09K1130A5R
- added U2: ICL7660M/TR, easyeda2kicad:SOP-8_L4.9-W3.9-P1.27-LS6.0-BL, symbol LCSC:ICL7660M_TR
- added U3: XC62KN3302PR-G, easyeda2kicad:SOT-89-3_L4.5-W2.5-P1.50-LS4.2-BR, symbol LCSC:XC62KN3302PR-G
- added U4: XC6206P332MR, easyeda2kicad:SOT-23-3_L2.9-W1.6-P1.90-LS2.8-BR, symbol LCSC:XC6206P332MR
- added U5: K7805M-1000R3_C41361052, easyeda2kicad:PWRM-TH_DEXU_K780XM-1000R3, symbol LCSC:K7805M-1000R3_C41361052
- J1: value Conn_01x02_Pin -> 9V_Bat
Connections:
- net 5V+: now also C2.1, C5.1, C7.1, U2.8 (V+), U4.3 (Vin), U5.3 (VOUT); no longer U1.2 (V-)
- net 5V-: now also C3.2, C9.2, U2.5 (VOUT), U3.1 (-VOUT); no longer U1.5 (V+)
- net GND: now also J1.9V- (Pin_2), C2.2, C3.1, C4.2, C5.2, C6.2, C7.2, C8.1, C9.1, CN1.1, U2.3 (GND), U2.6 (LV), U3.2 (VSS), U4.1 (GND), U5.2 (GND)
- net at R3.2: now also R5.3
- net SIG: now reaches U1.1 (OUTA)
- net SIG: now also R4.1, R5.2, R6.1
- new net: CN1.4, R6.2
- new net: CN1.3, R4.2
- new net: C1.1, U2.2 (CAP+)
- new net: C1.2, U2.4 (CAP–)
- new net: C4.1, J1.9V+ (Pin_1), U5.1 (VIN)
- new net 3V3+: C6.1, U1.5 (V+), U4.2 (Vout)
- new net 3V3-: C8.2, U1.2 (V-), U3.3 (-VIN)
- no-connect marks 0 -> 5
Other:
- moved on the sheet: J1, MK1, R1, R2, R3, U1
